File: Controller/My board_6.brd (EAGLE design)
At the start: 67.3 x 61.9 mm, 43 parts, among them J6 MALE 2x3, J7 POWER_JACKPTH_LOCK, U3 ATMEGA328, U4 FT232RLSSOP, X1 USB-B

Commit message: * Added LED to the control board for indicating that the OHC is sending a command * Corrections on the silkscreen for both boards (size of the names of the components)
Parts:
- removed LED4: Green, SparkFun:LED-0603
- added LED1: Green, LED:LED-0603
- added LED2: Red, SparkFun:LED-0603
- added R14: 1K, Passives:0603-RES
- J6: value MALE 2x3 -> ICSP
- J7: value POWER_JACKPTH_LOCK -> POWER_JACK
- JP2: device pinhead:1X06 -> con-samtec:TSW-106-02-S-S
- LED3: value Red -> Green
- U$1, U$2, U$3, U$4, U$9: value N-CHANNEL-MOSFET-BSS138 -> (none)
- U$10: value N-CHANNEL-MOSFET-BSS138 -> N-CHANNEL-MOSFETs-BSS138
- U4: value FT232RLSSOP -> FT232RL
- moved LED3 5.08 mm to (85.1, 30.5)
- turned JP2 to 0 degrees
Connections:
- new net S$4: R14.2, U3.1
- new net S$5: LED1.A, R14.1
- net GND: now also LED1.C
- net N$27: now also LED2.A; no longer LED3.A
- net N$28: now also LED3.A; no longer LED4.A
- net RXLED1: now also LED3.C; no longer LED4.C
- net TXLED1: now also LED2.C; no longer LED3.C
Routing:
- net S$4: track 0.00 -> 13.7 mm, vias 0 -> 2
- net GND: track 305.9 -> 312.4 mm
- net S$5: track 0.00 -> 2.72 mm
Other:
- board text added: "Designed by Eleftherios Nikolaidis"
