File: Controller/My board_6.sch (EAGLE design)
At the start: 43 parts, among them J6 MALE 2x3, J7 POWER_JACKPTH_LOCK, U3 ATMEGA328, U4 FT232RLSSOP, X1 USB-B

Commit message: * Added LED to the control board for indicating that the OHC is sending a command * Corrections on the silkscreen for both boards (size of the names of the components)
Parts:
- added LED1: Green, SparkFun:LED0603
- added R14: 1K, Passives:RESISTOR0603-RES
Connections:
- new net GND: J7.GND, J7.GNDBREAK, LED1.C
- new net N$11: LED1.A, R14.1
- new net N$12: R14.2, U3.PD3(INT1)
- net ASD: no longer J7.GND, J7.GNDBREAK
Other:
- moved on the sheet: C1, C13, C2, C3, C4, C5, C6, C7, J7, JP1, LED4, R13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
