File: LED_Board/LED_Board.sch (EAGLE design)
At the start: 16 parts

Commit message: * Added LED to the control board for indicating that the OHC is sending a command * Corrections on the silkscreen for both boards (size of the names of the components)
Parts:
- J1: value (none) -> +; device Connectors:M02PTH2 -> Connectors:M02LOCK
Other:
- moved on the sheet: J1
Changed lines of the file:
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@@
 <part name="R4" library="Passives" deviceset="RESISTOR" device="1206"/>
 <part name="R5" library="Passives" deviceset="RESISTOR" device="1206"/>
-<part name="J1" library="Connectors" deviceset="M02" device="PTH2"/>
+<part name="J1" library="Connectors" deviceset="M02" device="LOCK" value="+"/>
 <part name="LED2" library="led" deviceset="LED" device="5MM"/>
 <part name="LED3" library="led" deviceset="LED" device="5MM"/>
